File: PCB/AMD Challenge.kicad_pcb (KiCad board)
At the start: 2 copper layers, 53.5 x 70 mm, 9 parts, among them SW1 RotaryEncoder_Switch, SW2 SW_Push, SW3 SW_Push, U1 XIAO-RP2040-DIP

Commit message: Add files via upload
Parts:
- D1, D2, D3, D4: footprint LED_SMD:LED_SK6812MINI_PLCC4_3.5x3.5mm_P1.75mm -> footprints:SK6812MINI-E_fixed
- moved D2 1.85 mm to (239.5, 133.0)
Connections:
- D4 pad 1: Net-(D4-DOUT) -> unconnected-(D4-DOUT-Pad1)
Routing:
- net +5V: track 184.0 -> 223.8 mm, vias 2 -> 1
- net SK6812: track 52.4 -> 88.2 mm, vias 0 -> 1
- net GND: track 191.9 -> 209.6 mm, vias 0 -> 2
- net Net-(D2-DOUT): track 52.4 -> 40.6 mm
- net Net-(D3-DOUT): track 25.3 -> 36.1 mm, vias 0 -> 2
- net Net-(D1-DOUT): track 84.7 -> 87.6 mm, vias 0 -> 2
