File: PCB/AMD Challenge.kicad_sch (KiCad schematic)
At the start: 9 parts, among them SW1 RotaryEncoder_Switch, SW2 SW_Push, SW3 SW_Push, U1 XIAO-RP2040-DIP

Commit message: Add files via upload
Parts:
- D1, D2, D3, D4: footprint LED_SMD:LED_SK6812MINI_PLCC4_3.5x3.5mm_P1.75mm -> footprints:SK6812MINI-E_fixed
Changed lines of the file:
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@@
 			)
 		)
-		(property "Footprint" "LED_SMD:LED_SK6812MINI_PLCC4_3.5x3.5mm_P1.75mm"
+		(property "Footprint" "footprints:SK6812MINI-E_fixed"
 			(at 78.74 54.61 0)
 			(effects
@@
 			)
 		)
-		(property "Footprint" "LED_SMD:LED_SK6812MINI_PLCC4_3.5x3.5mm_P1.75mm"
+		(property "Footprint" "footprints:SK6812MINI-E_fixed"
 			(at 107.95 54.61 0)
 			(effects
@@
 			)
 		)
-		(property "Footprint" "LED_SMD:LED_SK6812MINI_PLCC4_3.5x3.5mm_P1.75mm"
+		(property "Footprint" "footprints:SK6812MINI-E_fixed"
 			(at 165.1 54.61 0)
 			(effects
@@
 			)
 		)
-		(property "Footprint" "LED_SMD:LED_SK6812MINI_PLCC4_3.5x3.5mm_P1.75mm"
+		(property "Footprint" "footprints:SK6812MINI-E_fixed"
 			(at 137.16 54.61 0)
 			(effects
